File: main.kicad_pcb (KiCad board)
At the start: 2 copper layers, 34.2 x 70.2 mm, 33 parts, among them J1 USB_A, J10 OrangePiCon, J2 USB_A, J3 USB_A, J4 USB_A, J5 USB_A, J6 Conn_01x02, J7 GS2, J8 GS2, U1 MIC5504-3.3YM5, U2 USB2514B_Bi, Y1 25MHz/50ppm

Commit message: Layout update
Parts:
- added C16: 100n, Capacitors_SMD:C_0603, B.Cu at (247.4, 146.8)
- J6: footprint Connectors_Terminal_Blocks:TerminalBlock_bornier-2_P5.08mm -> Pin_Headers:Pin_Header_Straight_1x02_Pitch2.54mm_SMD_Pin1Right
- J7, J8: moved to F.Cu
- Y1: footprint Oscillators:Oscillator_SMD_Abracon_ASE-4pin_3.2x2.5mm -> Crystals:Crystal_SMD_Abracon_ABM3-2pin_5.0x3.2mm
- moved C2 38.6 mm to (260.1, 154.9), turned to 0 degrees
- moved C1 37.0 mm to (259.6, 162.1), turned to 180 degrees
- moved U1 33.6 mm to (259.7, 158.1), turned to 90 degrees
- moved J6 32.0 mm to (258.6, 158.5), turned to 270 degrees
- moved J8 29.2 mm to (231.1, 162.1), turned to 90 degrees
- moved J1 24.8 mm to (246.4, 101.1), turned to 270 degrees
- moved J5 24.8 mm to (246.4, 118.9), turned to 270 degrees
- moved J3 24.0 mm to (251.1, 124.1), turned to 90 degrees
- moved J2 23.3 mm to (251.2, 141.6), turned to 90 degrees
- moved C7 18.7 mm to (259.6, 151.9)
- moved C3 18.7 mm to (254.0, 158.5), turned to 0 degrees
- moved C4 16.0 mm to (252.0, 147.5)
- moved R5 15.9 mm to (245.6, 146.9), turned to 90 degrees
- moved C6 15.6 mm to (261.1, 151.9), turned to 90 degrees
- moved C14 15.5 mm to (243.8, 146.9), turned to 270 degrees
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Connections:
- net USB1_DM renamed USB1-
- net USB1_DP renamed USB1+
- net USB2_DM renamed USB2-
- net USB2_DP renamed USB2+
- net USB3_DM renamed USB3-
- net USB3_DP renamed USB3+
- net USB4_DM renamed USB4-
- net USB4_DP renamed USB4+
- net USB5_DM renamed USB5-
- net USB5_DP renamed USB5+
- net USB_DM_UP renamed USB_UP-
- net USB_DP_UP renamed USB_UP+
Routing:
- net +3V3: track 0.00 -> 72.3 mm, vias 0 -> 6
- net +5V: track 0.00 -> 63.2 mm, vias 0 -> 5
- net USB1-: track 0.00 -> 51.3 mm
- net GND: track 60.5 -> 111.1 mm, vias 4 -> 1
- net USB1+: track 0.00 -> 46.7 mm
- net USB4+: track 0.00 -> 45.2 mm
- net USB4-: track 0.00 -> 45.0 mm
- net Net-(J10-Pad1): track 45.3 -> 2.68 mm
- net USB5-: track 36.2 -> 48.9 mm
- net Net-(J5-Pad5): track 12.0 -> 0.00 mm
- net USB2-: track 0.00 -> 11.7 mm
- net USB2+: track 0.00 -> 11.5 mm
- net USB3-: track 0.00 -> 10.4 mm
- net USB3+: track 0.00 -> 10.4 mm
- net USB5+: track 36.3 -> 46.6 mm
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- removed copper zone on B.Cu, net GND
- removed copper zone on F.Cu, net GND
Other:
- board size 34.2 x 70.2 mm -> 34.7 x 71.5 mm
- net class Power added: clearance 0.2, trace_width 0.5, via_dia 0.8, via_drill 0.4

Commit message: Layout draft 1
Parts:
- removed C11: 1uF, Capacitors_SMD:C_0603
- removed R2, R3: 100k, Resistors_SMD:R_0603
- removed R4: 1M, Resistors_SMD:R_0603
- moved R1 0.39 mm to (253.5, 160.8)
- moved C1 0.38 mm to (259.6, 161.7)
- moved C9 0.38 mm to (251.5, 161.2)
- moved Y1 0.38 mm to (244.7, 153.0)
Connections:
- J4 pad 5: Net-(J4-Pad5) -> GND
- J5 pad 5: Net-(J5-Pad5) -> GND
- U2 pad 27: Net-(R2-Pad1) -> +3V3
Routing:
- net GND: track 111.1 -> 239.6 mm, vias 1 -> 2
- net +5V: track 63.2 -> 115.2 mm, vias 5 -> 4
- net USB3+: track 10.4 -> 35.2 mm
- net USB3-: track 10.4 -> 33.8 mm
- net USB4+: track 45.2 -> 56.4 mm
- net USB4-: track 45.0 -> 55.7 mm
- net USB_UP+: track 8.34 -> 15.7 mm, vias 0 -> 1
- net Net-(R2-Pad1): track 5.99 -> 0.00 mm
- net USB2+: track 11.5 -> 17.4 mm
- net USB_UP-: track 8.71 -> 14.4 mm, vias 0 -> 1
- net USB2-: track 11.7 -> 16.0 mm
- net USB5-: track 48.9 -> 53.0 mm
- net Net-(C12-Pad1): track 9.73 -> 7.93 mm
- net Net-(C13-Pad1): track 9.58 -> 7.80 mm
- net +3V3: track 72.3 -> 73.1 mm, vias 6 -> 7
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- added copper zone on B.Cu, net GND
- added copper zone on F.Cu, net GND
